File: Add-OnV12.sch (EAGLE design)
At the start: 10 parts

Commit message: Update
Parts:
- removed IR1: TSOP1738TB1, telefunken:TSOP1738TB1
- removed U$1: TSOP1838, tsop-1:TSOP1838
- added SV1: (no value), con-lstb:MA04-1
- added X1: 1501_03, con-lumberg:1501_03
Connections:
- net GND: now also SV1.4, X1.1; no longer IR1.GND, U$1.GND
- net N$1: now also SV1.3, X1.3; no longer IR1.VS, U$1.V+
- net SCK: now also SV1.1, X1.2; no longer IR1.VO, U$1.OUT
Other:
- note added: "+"
- note added: "Achtung: PINS sind gespiegelt!"
- note added: "Out"
- note added: "TSOP1738TB1 (Beispiel)"
- note added: "laut VDR-Wiki: Basis -- GND Ring -- IR Tip -- VCC"
- note removed: "Achtung: PINS sind gespielt!"
Changed lines of the file:
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@@
 <parts>
 <part name="2USB-ASP" library="schwen" deviceset="CON2X5EDGE" device=""/>
-<part name="IR1" library="telefunken" deviceset="TSOP17*TB1" device="" technology="38"/>
 <part name="R1" library="rcl" deviceset="R-EU_" device="0204/2V" value="100"/>
 <part name="R2" library="rcl" deviceset="R-EU_" device="0204/2V" value="560"/>
@@
 <part name="SW" library="pinhead" deviceset="PINHD-1X2" device=""/>
 <part name="OK2" library="optocoupler" deviceset="PC817" device=""/>
-<part name="U$1" library="tsop-1" deviceset="TSOP1838" device=""/>
 <part name="GND4" library="supply1" deviceset="GND" device=""/>
+<part name="X1" library="con-lumberg" deviceset="1501_03" device=""/>
+<part name="SV1" library="con-lstb" deviceset="MA04-1" device=""/>
 </parts>
 <sheets>
 <sheet>
 <plain>
-<text x="-5.08" y="124.46" size="1.778" layer="91">Achtung: PINS sind gespielt!</text>
+<text x="-5.08" y="124.46" size="1.778" layer="91">Achtung: PINS sind gespiegelt!</text>
+<text x="-63.5" y="114.3" size="1.778" layer="91">Out</text>
+<text x="-63.5" y="119.38" size="1.778" layer="91">+</text>
+<text x="-99.06" y="134.62" size="1.778" layer="91">laut VDR-Wiki:
+Basis -- GND
+Ring -- IR
+Tip -- VCC</text>
+<text x="-73.66" y="104.14" size="1.778" layer="91">TSOP1738TB1
+(Beispiel)</text>
 </plain>
 <instances>
 <instance part="2USB-ASP" gate="G$1" x="10.16" y="111.76"/>
-<instance part="IR1" gate="A" x="-63.5" y="114.3"/>
 <instance part="R1" gate="G$1" x="-17.78" y="86.36"/>
 <instance part="R2" gate="G$1" x="-35.56" y="119.38"/>
@@
 <instance part="SW" gate="G$1" x="30.48" y="91.44" rot="R180"/>
 <instance part="OK2" gate="A" x="2.54" y="83.82"/>
-<instance part="U$1" gate="G$1" x="-66.04" y="134.62"/>
-<instance part="GND4" gate="1" x="-53.34" y="129.54" rot="R90"/>
+<instance part="GND4" gate="1" x="-45.72" y="139.7" rot="R90"/>
+<instance part="X1" gate="G$1" x="-76.2" y="137.16" rot="R180"/>
+<instance part="SV1" gate="1" x="-71.12" y="119.38"/>
 </instances>
 <busses>
@@
 <pinref part="C1" gate="G$1" pin="+"/>
 <wire x1="-45.72" y1="111.76" x2="-45.72" y2="119.38" width="0.1524" layer="91"/>
-<pinref part="IR1" gate="A" pin="VS"/>
-<wire x1="-45.72" y1="119.38" x2="-50.8" y2="119.38" width="0.1524" layer="91"/>
 <pinref part="R2" gate="G$1" pin="1"/>
 <wire x1="-40.64" y1="119.38" x2="-45.72" y2="119.38" width="0.1524" layer="91"/>
 <junction x="-45.72" y="119.38"/>
-<wire x1="-45.72" y1="119.38" x2="-45.72" y2="139.7" width="0.1524" layer="91"/>
-<pinref part="U$1" gate="G$1" pin="V+"/>
-<wire x1="-45.72" y1="139.7" x2="-58.42" y2="139.7" width="0.1524" layer="91"/>
+<pinref part="SV1" gate="1" pin="3"/>
+<wire x1="-45.72" y1="119.38" x2="-55.88" y2="119.38" width="0.1524" layer="91"/>
+<pinref part="X1" gate="G$1" pin="3"/>
+<wire x1="-55.88" y1="119.38" x2="-63.5" y2="119.38" width="0.1524" layer="91"/>
+<wire x1="-71.12" y1="134.62" x2="-55.88" y2="134.62" width="0.1524" layer="91"/>
+<wire x1="-55.88" y1="134.62" x2="-55.88" y2="119.38" width="0.1524" layer="91"/>
+<junction x="-55.88" y="119.38"/>
 </segment>
 </net>
 <net name="SCK" class="0">
 <segment>
-<pinref part="IR1" gate="A" pin="VO"/>
-<wire x1="-50.8" y1="114.3" x2="-48.26" y2="114.3" width="0.1524" layer="91"/>
 <label x="-5.08" y="114.3" size="1.778" layer="95"/>
-<pinref part="U$1" gate="G$1" pin="OUT"/>
-<wire x1="-58.42" y1="134.62" x2="-48.26" y2="134.62" width="0.1524" layer="91"/>
-<wire x1="-48.26" y1="134.62" x2="-48.26" y2="114.3" width="0.1524" layer="91"/>
-<junction x="-48.26" y="114.3"/>
 <pinref part="2USB-ASP" gate="G$1" pin="3"/>
-<wire x1="-48.26" y1="114.3" x2="5.08" y2="114.3" width="0.1524" layer="91"/>
+<wire x1="-63.5" y1="114.3" x2="-53.34" y2="114.3" width="0.1524" layer="91"/>
+<pinref part="SV1" gate="1" pin="1"/>
+<pinref part="X1" gate="G$1" pin="2"/>
+<wire x1="-53.34" y1="114.3" x2="5.08" y2="114.3" width="0.1524" layer="91"/>
+<wire x1="-71.12" y1="132.08" x2="-53.34" y2="132.08" width="0.1524" layer="91"/>
+<wire x1="-53.34" y1="132.08" x2="-53.34" y2="114.3" width="0.1524" layer="91"/>
+<junction x="-53.34" y="114.3"/>
 </segment>
 </net>
@@
 <pinref part="C1" gate="G$1" pin="-"/>
 <wire x1="-45.72" y1="104.14" x2="-50.8" y2="104.14" width="0.1524" layer="91"/>
-<pinref part="IR1" gate="A" pin="GND"/>
-<wire x1="-50.8" y1="104.14" x2="-50.8" y2="109.22" width="0.1524" layer="91"/>
 <pinref part="GND1" gate="1" pin="GND"/>
 <wire x1="-50.8" y1="99.06" x2="-50.8" y2="104.14" width="0.1524" layer="91"/>
-<junction x="-50.8" y="104.14"/>
 </segment>
 <segment>
@@
 <wire x1="-15.24" y1="76.2" x2="-15.24" y2="81.28" width="0.1524" layer="91"/>
 <wire x1="-15.24" y1="81.28" x2="-7.62" y2="81.28" width="0.1524" layer="91"/>
-</segment>
-<segment>
-<pinref part="U$1" gate="G$1" pin="GND"/>
-<wire x1="-58.42" y1="129.54" x2="-55.88" y2="129.54" width="0.1524" layer="91"/>
-<pinref part="GND4" gate="1" pin="GND"/>
 </segment>
 <segment>
@@
 <label x="17.78" y="111.76" size="1.778" layer="95"/>
 </segment>
+<segment>
+<pinref part="GND4" gate="1" pin="GND"/>
+<pinref part="X1" gate="G$1" pin="1"/>
+<wire x1="-48.26" y1="139.7" x2="-50.8" y2="139.7" width="0.1524" layer="91"/>
+<wire x1="-50.8" y1="139.7" x2="-71.12" y2="139.7" width="0.1524" layer="91"/>
+<wire x1="-50.8" y1="139.7" x2="-50.8" y2="121.92" width="0.1524" layer="91"/>
+<junction x="-50.8" y="139.7"/>
+<pinref part="SV1" gate="1" pin="4"/>
+<wire x1="-50.8" y1="121.92" x2="-63.5" y2="121.92" width="0.1524" layer="91"/>
+</segment>
 </net>
 <net name="N$3" class="0">
@@
 </sheet>
 </sheets>
-<errors>
-</errors>
 </schematic>
 </drawing>
+<compatibility>
+<note version="6.3" minversion="6.2.2" severity="warning">
+Since Version 6.2.2 text objects can contain more than one line,
+which will not be processed correctly with this version.
+</note>
+</compatibility>
 </eagle>
