File: Small/Add-OnV12.sch (EAGLE design)
At the start: 29 parts, among them IC1 MEGA48A-AU, K2 35701331, X1 1501_03

Commit message: Final Layout
Parts:
- removed C2: (no value), rcl:CPOL-EU085CS-1AR
- removed C3: 100n, rcl:C-EUC0805
- removed C4, C5: 22p, rcl:C-EUC0805
- removed CFG, OPT: (no value), con-lstb:MA03-2
- removed D1, D2: 3V6, diode:ZENER-DIODESOD80C
- removed IC1: MEGA48A-AU, atmel:MEGA8-AI
- removed IR, MB-SW: (no value), con-lstb:MA04-1
- removed ISP: (no value), con-lstb:MA05-2
- removed K2: 35701331, relay:35701331
- removed LED1: green, led:LEDCHIPLED_1206
- removed LED2: red, led:LEDCHIPLED_1206
- removed OK1: PC817, optocoupler:PC817
- removed Q2: (no value), crystal:CRYSTALHC49UP
- removed R3: 2k2, rcl:R-EU_M0805
- removed R4, R5, R7: 1k, rcl:R-EU_M0805
- removed R6: 10k, rcl:R-EU_M0805
- removed R8, R9: 560, rcl:R-EU_M0805
- removed SV2: (no value), con-lsta:FE05W
- added 2USB-ASP: CON2X5EDGE, schwen:CON2X5EDGE
- added FREI: (no value), con-lstb:MA03-1
- added MB, SW: (no value), pinhead:PINHD-1X2
- added OK2: PC817, optocoupler:PC817
- added SV1: (no value), con-lstb:MA04-1
- C1: value 4u7 -> 4,7uF; device rcl:C-EUC0805 -> rcl:CPOL-EUE1.8-4
- R1: value 68 -> 100; device rcl:R-EU_M0805 -> rcl:R-EU_0204/2V
- R2: value 68 -> 560; device rcl:R-EU_M0805 -> rcl:R-EU_0204/2V
Connections:
- removed net +5V: C1.1, C3.1, CFG.5, CFG.6, IC1.AVCC, IC1.VCC@1, IC1.VCC@2, ISP.2, R3.1, R4.1, R5.1, R6.1, R8.2, SV2.1
- removed net ADC6: IC1.ADC6
- removed net D+: D1.C, R2.1, SV2.3
- removed net D-: D2.C, R1.1, R3.2, SV2.2
- removed net N$13: LED2.A, R4.2
- removed net N$14: IC1.PC0(ADC0), LED2.C
- removed net N$15: IC1.PC1(ADC1), LED1.C
- removed net N$16: IC1.PB0(ICP), R1.2
- removed net N$21: IC1.PD3(INT1)
- removed net N$22: C4.2, IC1.PB6(XTAL1/TOSC1), Q2.1
- removed net N$23: C5.2, IC1.PB7(XTAL2/TOSC2), Q2.2
- removed net N$25: LED1.A, R5.2
- removed net N$6: IC1.PD1(TXD), R7.2
- removed net N$7: IC1.PB1(OC1A), IC1.PD2(INT0), R2.2
- removed net PB2-RST: CFG.2, IC1.PB2(SS/OC1B), ISP.5
- removed net PC3: IC1.PC3(ADC3), OPT.4
- removed net PC4: IC1.PC4(ADC4/SDA), OPT.1
- removed net PC5: IC1.PC5(ADC5/SCL)
- removed net PD4: IC1.PD4(XCK/T0), OPT.3
- removed net PD5: IC1.PD5(T1), OPT.2
- removed net PD6: IC1.PD6(AIN0), OPT.6
- removed net PD7: IC1.PD7(AIN1), OPT.5
- removed net RX: IC1.PD0(RXD), ISP.6
- removed net SW1: K22.P, MB-SW.1, MB-SW.4, OK1.COL
- removed net SW2: K22.S, MB-SW.2, MB-SW.3, OK1.EMIT
- removed net TX: ISP.4, R7.1
- new net N$3: MB.2, OK2.COL, SW.1
- new net NC: 2USB-ASP.7, FREI.2
- new net VCC: 2USB-ASP.10, R2.2
- net GND: now also 2USB-ASP.2, 2USB-ASP.4, 2USB-ASP.6, 2USB-ASP.8, C1.-, OK2.C, SV1.4; no longer C1.2, C2.-, C3.2, C4.1, C5.1, CFG.4, D1.A, D2.A, IC1.AGND, IC1.GND@1, IC1.GND@2, IR.1, ISP.10, ISP.8, K21.5, OK1.C, SV2.4
- net MISO: now also 2USB-ASP.1, R1.1; no longer IC1.PB4(MISO), ISP.9, K21.3, R9.2
- net MOSI: now also 2USB-ASP.9, FREI.1; no longer IC1.PB3(MOSI/OC2), ISP.1
- net N$1: now also C1.+, R2.1, SV1.3, X1.3; no longer OK1.A, R9.1
- net N$2: now also OK2.A, R1.2; no longer CFG.3, IC1.PC2(ADC2)
- net N$4: now also MB.1, OK2.EMIT, SW.2; no longer C2.+, IR.2, R8.1, X1.3
- net RST: now also 2USB-ASP.5, FREI.3; no longer CFG.1, IC1.PC6(/RESET), R6.2
- net SCK: now also 2USB-ASP.3, SV1.1; no longer IC1.PB5(SCK), IR.4, ISP.7
Other:
- note added: "+"
- note added: "Achtung: PINS sind gespiegelt!"
- note added: "Out"
- note added: "TSOP1738TB1 (Beispiel)"
- note added: "laut VDR-Wiki: Basis -- GND Ring -- IR Tip -- VCC"
- note removed: "*) ATMEGA 168A-AU, Mega48 or Mega8"
- note removed: "Basis: http://www.fischl.de/usbasp/"
- note removed: "SIL 7271-D 5V"
- moved on the sheet: R1, R2, X1
